File: moodlight.sch (KiCad schematic (older format))
At the start: 40 parts, among them IC1 AT90USB16, Q1 BC847C, Q2 BC847C, Q3 BC847C, SW1 SWITCH_PUSHBUTTON, SW2 SWITCH_PUSHBUTTON, U1 USBCONN, X1 16MHz

Commit message: MoodLight V2 - changed pins: R = 21, G = 23, B = 25 - no quartz - different ESDs (SOT23EBC body) - different LEDs (PCC6 5050) - slightly adapted shape to fit the lampions more easily
Parts:
- removed C3, C7: 18p, symbol C_MINI
- removed CR1, CR2: ESD_Zener, symbol ESD_Zener
- removed LED1, LED2, LED3, LED4: LED_RCBG, symbol LED_RCBG
- removed X1: 16MHz, symbol CRYSTAL
- added D1, D2, D3, D4: IMPOLUX_RGB_SMD, symbol IMPOLUX_RGB_SMD
- added ESD1: ESD_TWO-LINE, symbol ESD_TWO-LINE
Connections:
- wire segments 112 -> 116
- no-connect marks 17 -> 19
Other:
- moved on the sheet: C1, C2, C4, C5, C6, SW1, SW2, U1

Commit message: Di 29. Okt 15:49:31 CET 2013
Parts:
- added C7, C8: 12pF, ~, symbol CP1
- added P1: CONN_8X2, ~, symbol CONN_8X2
- added X1: CRYSTAL, ~, symbol CRYSTAL
Connections:
- net labels added: PB0, PB1, PB2, PB3, PB4, PB5, PB6, PD0, PD1, PD2, PD3, PD4, PD5, PD6
- wire segments 116 -> 154
- no-connect marks 19 -> 3
Other:
- moved on the sheet: C1, C2
