File: moodlight.sch (KiCad schematic (older format))
At the start: 40 parts, among them IC1 AT90USB16, P1 CONN_8X2, Q1 BC847C, Q2 BC847C, Q3 BC847C, SW1 SWITCH_PUSHBUTTON, SW2 SWITCH_PUSHBUTTON, U1 USBCONN, X1 CRYSTAL

Commit message: Mi 30. Okt 20:03:15 CET 2013
Parts:
- added P?: CONN_5X2, symbol CONN_5X2
Changed lines of the file:
@@
 $EndComp
 $Comp
-L VCC #PWR?
+L VCC #PWR036
 U 1 1 51DEF637
 P 4900 6200
-F 0 "#PWR?" H 4900 6300 30  0001 C CNN
+F 0 "#PWR036" H 4900 6300 30  0001 C CNN
 F 1 "VCC" H 4900 6300 30  0000 C CNN
 F 2 "" H 4900 6200 60  0001 C CNN
@@
 $EndComp
 $Comp
-L GND #PWR?
+L GND #PWR037
 U 1 1 51DEF63D
 P 5650 5950
-F 0 "#PWR?" H 5650 5950 30  0001 C CNN
+F 0 "#PWR037" H 5650 5950 30  0001 C CNN
 F 1 "GND" H 5650 5880 30  0001 C CNN
 F 2 "" H 5650 5950 60  0001 C CNN
@@
 Wire Wire Line
 	6100 6900 5850 6900
+$Comp
+L CONN_5X2 P?
+U 1 1 527118BC
+P 5450 5400
+F 0 "P?" H 5450 5700 60  0000 C CNN
+F 1 "CONN_5X2" V 5450 5400 50  0000 C CNN
+F 2 "" H 5450 5400 60  0000 C CNN
+F 3 "" H 5450 5400 60  0000 C CNN
+	1    5450 5400
+	1    0    0    -1
+$EndComp
 $EndSCHEMATC

Commit message: v3 first prototype
Parts:
- removed C1, C2: 0u1, symbol C_MINI
- removed P?: CONN_5X2, symbol CONN_5X2
Connections:
- wire segments 154 -> 150
Changed lines of the file:
@@
 LIBS:Micropendous-32U2-cache
 LIBS:LED_RGB
-LIBS:moodlight-cache
 EELAYER 24 0
 EELAYER END
@@
 Wire Wire Line
 	3400 5000 3400 5050
-Wire Wire Line
-	950  4000 950  3900
-Wire Wire Line
-	750  3700 750  3600
 Connection ~ 5150 4000
 Wire Wire Line
@@
 Wire Wire Line
 	3400 6150 3400 6200
-Wire Wire Line
-	950  3700 950  3600
-Wire Wire Line
-	750  4000 750  3900
 Wire Wire Line
 	3400 5700 3400 5750
@@
 	1    8350 2750
 	0    -1   -1   0
-$EndComp
-$Comp
-L GND #PWR014
-U 1 1 4E2744FB
-P 950 4000
-F 0 "#PWR014" H 950 4000 30  0001 C CNN
-F 1 "GND" H 950 3930 30  0001 C CNN
-F 2 "" H 950 4000 60  0001 C CNN
-F 3 "" H 950 4000 60  0001 C CNN
-	1    950  4000
-	1    0    0    -1
-$EndComp
-$Comp
-L GND #PWR015
-U 1 1 4E2744ED
-P 750 4000
-F 0 "#PWR015" H 750 4000 30  0001 C CNN
-F 1 "GND" H 750 3930 30  0001 C CNN
-F 2 "" H 750 4000 60  0001 C CNN
-F 3 "" H 750 4000 60  0001 C CNN
-	1    750  4000
-	1    0    0    -1
-$EndComp
-$Comp
-L VDD #PWR016
-U 1 1 4E2744C4
-P 750 3600
-F 0 "#PWR016" H 750 3700 30  0001 C CNN
-F 1 "VDD" H 750 3710 30  0000 C CNN
-F 2 "" H 750 3600 60  0001 C CNN
-F 3 "" H 750 3600 60  0001 C CNN
-	1    750  3600
-	1    0    0    -1
-$EndComp
-$Comp
-L VCC #PWR017
-U 1 1 4E2744BD
-P 950 3600
-F 0 "#PWR017" H 950 3700 30  0001 C CNN
-F 1 "VCC" H 950 3700 30  0000 C CNN
-F 2 "" H 950 3600 60  0001 C CNN
-F 3 "" H 950 3600 60  0001 C CNN
-	1    950  3600
-	1    0    0    -1
-$EndComp
-$Comp
-L C_MINI C1
-U 1 1 4E2744B3
-P 750 3800
-F 0 "C1" V 700 3840 30  0000 C CNN
-F 1 "0u1" V 800 3870 25  0000 C CNN
-F 2 "" H 750 3800 60  0001 C CNN
-F 3 "" H 750 3800 60  0001 C CNN
-	1    750  3800
-	0    1    1    0
-$EndComp
-$Comp
-L C_MINI C2
-U 1 1 4E2744A8
-P 950 3800
-F 0 "C2" V 900 3840 30  0000 C CNN
-F 1 "0u1" V 1000 3870 25  0000 C CNN
-F 2 "" H 950 3800 60  0001 C CNN
-F 3 "" H 950 3800 60  0001 C CNN
-	1    950  3800
-	0    1    1    0
 $EndComp
 $Comp
@@
 Wire Wire Line
 	6100 6900 5850 6900
-$Comp
-L CONN_5X2 P?
-U 1 1 527118BC
-P 5450 5400
-F 0 "P?" H 5450 5700 60  0000 C CNN
-F 1 "CONN_5X2" V 5450 5400 50  0000 C CNN
-F 2 "" H 5450 5400 60  0000 C CNN
-F 3 "" H 5450 5400 60  0000 C CNN
-	1    5450 5400
-	1    0    0    -1
-$EndComp
 $EndSCHEMATC

Commit message: Removed ESD Diodes. Footprints etc. appear to be correct now.
Parts:
- removed ESD1: ESD_TWO-LINE, symbol ESD_TWO-LINE
Connections:
- wire segments 150 -> 146
Changed lines of the file:
@@
 LIBS:Micropendous-32U2-cache
 LIBS:LED_RGB
+LIBS:w_opto
+LIBS:moodlight-cache
+LIBS:moodlight-cache
 EELAYER 24 0
 EELAYER END
@@
 Comment4 ""
 $EndDescr
-Connection ~ 4650 3500
-Wire Wire Line
-	4650 3800 4650 3500
 Wire Wire Line
 	4850 3600 4850 3500
 Wire Wire Line
 	4300 3600 4850 3600
-Connection ~ 4350 3600
-Wire Wire Line
-	4350 3800 4350 3600
-Connection ~ 4500 4250
 Wire Wire Line
 	8600 2450 8950 2450
@@
 	10450 6650 10450 6700
 Wire Wire Line
-	5150 3500 5150 4250
-Wire Wire Line
-	4500 4350 4500 4200
-Wire Wire Line
-	5150 4250 4500 4250
-Wire Wire Line
 	4750 3500 4300 3500
 $Comp
 L GND #PWR01
 U 1 1 4F6F8E71
-P 4500 4350
-F 0 "#PWR01" H 4500 4350 30  0001 C CNN
-F 1 "GND" H 4500 4280 30  0001 C CNN
-F 2 "" H 4500 4350 60  0001 C CNN
-F 3 "" H 4500 4350 60  0001 C CNN
-	1    4500 4350
-	1    0    0    -1
-$EndComp
-$Comp
-L ESD_TWO-LINE ESD1
-U 1 1 4F6F8DFD
-P 4550 4250
-F 0 "ESD1" V 4250 4500 60  0000 C CNN
-F 1 "ESD_TWO-LINE" V 4750 4550 60  0000 C CNN
-F 2 "" H 4550 4250 60  0001 C CNN
-F 3 "" H 4550 4250 60  0001 C CNN
-	1    4550 4250
+P 5150 4200
+F 0 "#PWR01" H 5150 4200 30  0001 C CNN
+F 1 "GND" H 5150 4130 30  0001 C CNN
+F 2 "" H 5150 4200 60  0001 C CNN
+F 3 "" H 5150 4200 60  0001 C CNN
+	1    5150 4200
 	1    0    0    -1
 $EndComp
@@
 Wire Wire Line
 	6100 6900 5850 6900
+Wire Wire Line
+	5150 3500 5150 4200
 $EndSCHEMATC
